File: Ghost32.kicad_pcb (KiCad board)
At the start: 4 copper layers, 102.5 x 100.8 mm, 88 parts, among them J1 USB_C_Receptacle_USB2.0_16P, J10 Motor 3, J11 Power Input L293d, J12 Motor 3, J2 USB_C_Receptacle_USB2.0_16P, J3 Conn_01x09_Socket, J4 Conn_01x15_Socket, J5 Conn_01x09_Socket, J6 ESP32_Socket_2, J7 Motor 1, J8 Motor 2, J9 Conn_01x13_Socket, SW1 SW_Push, SW2 SW_Push, SW3 SW_DIP_x01, SW4 SW_DIP_x01, SW5 Boot, SW6 Reset, U1 TB6612FNG, U2 ESP32-S3-MINI-1, U3 MPU-6050, U5 AP2112K-3.3, U6 RP2350_60QFN, U7 TB6612FNG, U8 W25Q64JVXGIQ TR, Y1 ABM8-272-T3

Commit message: Update Ghost32.kicad_pcb
Routing:
- net +1V1: track 39.0 -> 38.0 mm
Changed lines of the file:
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@@
+	)
+	(segment
+		(start 165.710823 133.339998)
+		(end 165.710823 133.255569)
+		(width 0.2)
+		(layer "F.Cu")
+		(net 6)
 	)
 	(segment
@@
 	)
 	(segment
-		(start 165.23 133.08)
-		(end 165.15 133.16)
-		(width 0.2)
-		(layer "F.Cu")
-		(net 6)
-	)
-	(segment
 		(start 156.800589 131.540589)
 		(end 156.860589 131.540589)
@@
 		(start 168.81245 124.12)
 		(end 166.62 126.31245)
-		(width 0.2)
-		(layer "F.Cu")
-		(net 6)
-	)
-	(segment
-		(start 165.55 133.08)
-		(end 165.37 133.08)
 		(width 0.2)
 		(layer "F.Cu")
@@
 	)
 	(segment
-		(start 165.82 132.09)
-		(end 165.82 133.08)
+		(start 165.710823 133.255569)
+		(end 165.82 133.146392)
 		(width 0.2)
 		(layer "F.Cu")
@@
 		(start 167.05 134.99)
 		(end 167.04 134.98)
-		(width 0.2)
-		(layer "F.Cu")
-		(net 6)
-	)
-	(segment
-		(start 165.55 133.08)
-		(end 165.23 133.08)
 		(width 0.2)
 		(layer "F.Cu")
@@
 	)
 	(segment
-		(start 165.82 133.08)
-		(end 165.55 133.08)
-		(width 0.2)
-		(layer "F.Cu")
-		(net 6)
-	)
-	(segment
 		(start 166.08 130.97)
 		(end 166.516373 130.533627)
@@
 	)
 	(segment
+		(start 165.82 133.146392)
+		(end 165.82 132.09)
+		(width 0.2)
+		(layer "F.Cu")
+		(net 6)
+	)
+	(segment
 		(start 166.62 127.32)
 		(end 167.51 127.32)
@@
 	)
 	(segment
-		(start 165.82 133.08)
-		(end 165.83 133.09)
-		(width 0.2)
-		(layer "F.Cu")
-		(net 6)
-	)
-	(segment
 		(start 166.62 126.31245)
 		(end 166.62 127.32)
@@
 	)
 	(via
+		(at 165.710823 133.339998)
+		(size 0.6)
+		(drill 0.3)
+		(layers "F.Cu" "B.Cu")
+		(net 6)
+	)
+	(via
 		(at 166.62 127.32)
 		(size 0.6)
@@
 	(via
 		(at 156.28 134.44)
-		(size 0.6)
-		(drill 0.3)
-		(layers "F.Cu" "B.Cu")
-		(net 6)
-	)
-	(via
-		(at 165.15 133.16)
 		(size 0.6)
 		(drill 0.3)
@@
 	)
 	(segment
+		(start 166.97 134.98)
+		(end 167.04 134.98)
+		(width 0.2)
+		(layer "In2.Cu")
+		(net 6)
+	)
+	(segment
 		(start 163.480617 132.989326)
 		(end 166.516373 129.95357)
@@
 	)
 	(segment
+		(start 165.673503 133.683503)
+		(end 166.97 134.98)
+		(width 0.2)
+		(layer "In2.Cu")
+		(net 6)
+	)
+	(segment
 		(start 160.231826 134.168174)
 		(end 161.410674 132.989326)
@@
 	)
 	(segment
-		(start 165.15 133.16)
-		(end 166.97 134.98)
-		(width 0.2)
-		(layer "In2.Cu")
-		(net 6)
-	)
-	(segment
 		(start 161.410674 132.989326)
 		(end 163.480617 132.989326)
@@
 	)
 	(segment
-		(start 166.97 134.98)
-		(end 167.04 134.98)
-		(width 0.2)
-		(layer "In2.Cu")
+		(start 165.710823 133.339998)
+		(end 165.673503 133.377318)
+		(width 0.2)
+		(layer "In2.Cu")
+		(net 6)
+	)
+	(segment
+		(start 165.673503 133.377318)
+		(end 165.673503 133.683503)
+		(width 0.2)
+		(layer "In2.Cu")
